Commit message: Gazebo simulation

File: src/arduinobot_description/urdf/arduinobot.urdf.xacro (robot description, xacro)
@@ -122,4 +122,60 @@
         </collision>
     </link>
+    <!-- Add camera-->
+    <link name="rgb_camera">
+        <visual>
+            <xacro:default_inertial mass="0.001"/>
+            <origin rpy="-1.57 0 -1.57" xyz="-0.05 0.122 0.14"/>
+            <geometry>
+                <mesh filename="package://arduinobot_description/meshes/pi_camera.STL" scale="0.01 0.01 0.01"/>
+            </geometry>
+        </visual>
+        <collision>
+            <origin rpy="-1.57 0 -1.57" xyz="-0.05 0.122 0.14"/>
+            <geometry>
+                <mesh filename="package://arduinobot_description/meshes/pi_camera.STL" scale="0.01 0.01 0.01"/>
+            </geometry>
+        </collision>
+    </link>
+    <joint name="rgb_camera_joint" type="fixed">
+        <parent link="base_link"/>
+        <child link="rgb_camera"/>
+        <origin xyz="0 0.45 0.2" rpy="0 -0.5 1.57"/>
+    </joint>
+    <gazebo reference="rgb_camera">
+        <sensor name="camera" type="camera">
+            <always_on>true</always_on>
+            <update_rate>30.0</update_rate>
+            <visualize>true</visualize>
+            <topic>/image_raw</topic>
+            <gz_frame_id>/rgb_camera</gz_frame_id>
+            <camera name="camera">
+              <horizontal_fov>1.21126</horizontal_fov>
+              <image>
+                <width>2304</width>
+                <height>1296</height>
+                <format>R8G8B8</format>
+              </image>
+              <distortion>
+                <k1>0.0</k1>
+                <k2>0.0</k2>
+                <k3>0.0</k3>
+                <p1>0.0</p1>
+                <p2>0.0</p2>
+                <center>0.5 0.5</center>
+              </distortion>
+            </camera>
+        </sensor>
+        <plugin name="camera_plugin" filename="libgazebo_ros_camera.so">
+            <ros>
+                <!-- Option A: Directly rename the camera_name -->
+                <!-- <namespace>rgb_camera</namespace> -->
+                <remapping>~/image_raw:=image_raw</remapping>
+                <remapping>~/camera_info:=camera_info</remapping>
+            </ros>
+            <camera_name>rgb_camera</camera_name>
+            <frame_name>rgb_camera</frame_name>
+        </plugin>
+    </gazebo>
     <!-- Joints -->
     <joint name="virtual_joint" type="fixed">
